Commit message: Updated to allow multiple IMU sensors on the same CAN bus. Attempted to keep the structure the same by having a lookup map for the frame_id switch case:
1) Added param for CAN interface
2) Added params to define each frame id in the yaml file. These should be defined to match the frames the xsens imu is configured to send.
3) Added socket CAN filter to filter only the frame ids defined in the yaml file, to reduce node processing on full can buses
4) Altered error checking on the socket connection and bind and close the ros node

File: src/xsens_mti_can_ros_driver/urdf/MTi_1.urdf (robot description, URDF)
Before this commit: robot mti_1, 1 links, 0 joints
Links:
- link imu_link: geometry visual mesh filename=package://xsens_mti_can_ros_driver/urdf/MTi_1.stl scale=0.001 0.001 0.001

File: src/xsens_mti_can_ros_driver/urdf/MTi_10.urdf (robot description, URDF)
Before this commit: robot mti_10, 1 links, 0 joints
Links:
- link imu_link: geometry visual mesh filename=package://xsens_mti_can_ros_driver/urdf/MTi_10.stl scale=0.001 0.001 0.001

File: src/xsens_mti_can_ros_driver/urdf/MTi_6xx.urdf (robot description, URDF)
Before this commit: robot mti_6xx, 1 links, 0 joints
Links:
- link imu_link: geometry visual mesh filename=package://xsens_mti_can_ros_driver/urdf/MTi_6xx.stl scale=0.001 0.001 0.001
